Commit message: 9.1完成到上实机之前，最后检查安全性

File: vr_rm75_ws/install/lsrx_rm75_dual_description/share/lsrx_rm75_dual_description/urdf/LSRX_RM75_DUAL.urdf (robot description, URDF)
Before this commit: robot LSRX_RM75_DUAL, 59 links, 58 joints
Joints:
- joint l_rm75_camera_joint: origin xyz=0.029031 -0.10022 -0.0005 rpy=0 1.5708 0 -> xyz=0.029031 -0.10022 0.0005 rpy=0 1.5707963268 0
- joint l_rm75_camera_rojoint: axis 0 0 1 -> (none); limit lower=0 upper=1.05 effort=0 velocity=0 -> (none); origin xyz=0.033 -0.0085 -0.05388 rpy=1.5708 1.5708 3.1416 -> xyz=-0.033 0.0085 -0.05388 rpy=-1.5707963268 -1.5707963268 0; type revolute -> fixed
